Commit message: Fix warnings in Jade

File: hilgendorf_support/urdf/hilgendorf.xacro (robot description, xacro)
@@ -1,4 +1,4 @@
 <?xml version="1.0"?>
-<robot xmlns:xacro="http://www.ros.org/wiki/xacro"
+<robot xmlns:xacro="http://ros.org/wiki/xacro"
        name="hilgendorf" >
   <xacro:include filename="$(find hilgendorf_support)/urdf/hilgendorf_macro.xacro" />

File: hilgendorf_support/urdf/hilgendorf_base_macro.xacro (robot description, xacro)
@@ -7,9 +7,9 @@
     Left Arm: "[prefix]left_shoulder"
  -->
-<robot xmlns:xacro="http://www.ros.org/wiki/xacro">
+<robot xmlns:xacro="http://ros.org/wiki/xacro">
   <!-- Physical dimensions of the base -->
-  <property name="base_shoulder_height" value="0.54" />
-  <property name="base_shoulder_width" value="0.665" />
-  <property name="base_shoulder_angle" value="2.356194490192345" />
+  <xacro:property name="base_shoulder_height" value="0.54" />
+  <xacro:property name="base_shoulder_width" value="0.665" />
+  <xacro:property name="base_shoulder_angle" value="2.356194490192345" />
   <!-- Base macro -->
   <xacro:macro name="hilgendorf_base" params="prefix">

File: hilgendorf_support/urdf/hilgendorf_macro.xacro (robot description, xacro)
@@ -1,5 +1,5 @@
 <?xml version="1.0"?>
 <!-- URDF-XACRO file for generating a Hilgendorf dual-arm robot-->
-<robot xmlns:xacro="http://www.ros.org/wiki/xacro">
+<robot xmlns:xacro="http://ros.org/wiki/xacro">
   <!-- base -->
   <xacro:include filename="$(find hilgendorf_support)/urdf/hilgendorf_base_macro.xacro" />
@@ -9,6 +9,6 @@
   <xacro:include filename="$(find robotiq_c2_model_visualization)/urdf/robotiq_c2_model_macro.xacro" />
   <!-- Physical dimensions -->
-  <property name="ur5_mount_angle_offset" value="-0.7853981633974483" />
-  <property name="robotiq_grip_target_offset" value="0.1" />
+  <xacro:property name="ur5_mount_angle_offset" value="-0.7853981633974483" />
+  <xacro:property name="robotiq_grip_target_offset" value="0.1" />
   <xacro:macro name="hilgendorf" params="prefix">
     <!-- Arm mount -->
